File: pcb/choctopus44.kicad_pcb (KiCad board)
At the start: 2 copper layers, 243.9 x 111.9 mm, 110 parts, among them SW1 SW_PUSH, SW10 SW_PUSH, SW11 SW_PUSH, SW12 SW_PUSH, SW13 SW_PUSH, SW14 SW_PUSH, SW15 SW_PUSH, SW16 SW_PUSH, SW17 SW_PUSH, SW18 SW_PUSH, SW19 SW_PUSH, SW2 SW_PUSH, SW20 SW_PUSH, SW21 SW_PUSH, SW22 SW_PUSH, SW23 SW_PUSH, SW24 SW_PUSH, SW25 SW_PUSH, SW26 SW_PUSH, SW27 SW_PUSH, SW28 SW_PUSH, SW29 SW_PUSH, SW3 SW_PUSH, SW30 SW_PUSH, SW31 SW_PUSH, SW32 SW_PUSH, SW33 SW_PUSH, SW34 SW_PUSH, SW35 SW_PUSH, SW36 SW_PUSH, SW37 SW_PUSH, SW38 SW_PUSH, SW39 SW_PUSH, SW4 SW_PUSH, SW40 SW_PUSH, SW41 SW_PUSH, SW42 SW_PUSH, SW43 SW_PUSH, SW44 SW_PUSH, SW45 Rotary_Encoder_Switch, SW5 SW_PUSH, SW6 SW_PUSH, SW7 SW_PUSH, SW8 SW_PUSH, SW9 SW_PUSH, U1 ProMicro

Commit message: Sorted some Error
Parts:
- removed RESET1: SW_PUSH, Button_Switch_THT:SW_TH_Tactile_Omron_B3F-10xx
- removed SW_PWR1: SW_DPST, Button_Switch_THT:SW_E-Switch_EG1271_DPDT
- added SW46: SW_Push_DPDT, Button_Switch_THT:SW_E-Switch_EG1271_DPDT, F.Cu at (173.1, 65.5)
- added SW47: SW_SPST, Button_Switch_THT:SW_TH_Tactile_Omron_B3F-10xx, F.Cu at (169.3, 61.0)
Routing:
- net Net-(BT1-Pad2): track 21.0 -> 16.7 mm
- net +BATT: track 53.3 -> 56.5 mm
- net Net-(BT1-Pad1): track 17.1 -> 16.3 mm, vias 0 -> 1
