File: kicad/ver1.0 RC-1/pcb/choctopus44.kicad_sch (KiCad schematic)
At the start: 103 parts, among them SW1 SW_PUSH, SW10 SW_PUSH, SW11 SW_PUSH, SW12 SW_PUSH, SW13 SW_PUSH, SW14 SW_PUSH, SW15 SW_PUSH, SW16 SW_PUSH, SW17 SW_PUSH, SW18 SW_PUSH, SW19 SW_PUSH, SW2 SW_PUSH, SW20 SW_PUSH, SW21 SW_PUSH, SW22 SW_PUSH, SW23 SW_PUSH, SW24 SW_PUSH, SW25 SW_PUSH, SW26 SW_PUSH, SW27 SW_PUSH, SW28 SW_PUSH, SW29 SW_PUSH, SW3 SW_PUSH, SW30 SW_PUSH, SW31 SW_PUSH, SW32 SW_PUSH, SW33 SW_PUSH, SW34 SW_PUSH, SW35 SW_PUSH, SW36 SW_PUSH, SW37 SW_PUSH, SW38 SW_PUSH, SW39 SW_PUSH, SW4 SW_PUSH, SW40 SW_PUSH, SW41 SW_PUSH, SW42 SW_PUSH, SW43 SW_PUSH, SW44 SW_PUSH, SW45_2 SW_PUSH, SW5 SW_PUSH, SW6 SW_PUSH, SW7 SW_PUSH, SW8 SW_PUSH, SW9 SW_PUSH, U1 ProMicro

Commit message: backups etc
Parts:
- added NT1: NetTie_2, symbol Device:NetTie_2
- SW45: renamed from SW?; symbol Device:Rotary_Encoder_Switch -> Device:RotaryEncoder_Switch
- U1: value ProMicro -> ProMicro/Nice!Nano; footprint Keebio-Parts:ArduinoProMicro -> promicro-nicenano:promicro-nicenano; symbol choctopus44-rescue:ProMicro-_reviung-kbd-reviung41-rescue -> promicro-nicenano:promicro-nicenano
- gave numbers to parts that had none: 8
Connections:
- net GND: now also U1.14 (GND), NT1.1; no longer U1.23 (GND)
- net VCC: now also U1.16 (VCC); no longer U1.21 (VCC)
- net reset: now also U1.15 (RST); no longer U1.22 (RST)
- net row0: now also U1.17 (F4); no longer U1.20 (F4/A3)
- net row1: now also U1.18 (F5); no longer U1.19 (F5/A2)
- net row2: now also U1.19 (F6); no longer U1.18 (F6/A1)
- net row3: now also U1.20 (F7); no longer U1.17 (F7/A0)
- net row4: now also U1.21 (B1); no longer U1.16 (B1/15)
- net row5: now also U1.22 (B3); no longer U1.15 (B3/14)
- net row6: now also U1.23 (B2); no longer U1.14 (B2/16)
- net at SW_PWR1.2: now also BT1.1 (+); no longer BT1.2 (-)
- net at SW_PWR1.4: now also BT1.2 (-); no longer BT1.1 (+)
- net +BATT: no longer names the net of SW_PWR1.1
- net +BATT: now also U1.26 (B+)
- net -BATT: no longer names the net of SW_PWR1.3
- net -BATT: now also U1.25 (GND/B-), NT1.2
Other:
- moved on the sheet: BT1, SW_PWR1

Commit message: Schema done, PCB work restarted
Parts:
- NT1: footprint (none) -> NetTie:NetTie-2_SMD_Pad0.5mm
- SW45: footprint Rotary_Encoder:RotaryEncoder_Alps_EC11E-Switch_Vertical_H20mm-SMD-support -> Rotary_Encoder:RotaryEncoder_Alps_EC11E-Switch_Vertical_H20mm
Changed lines of the file:
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@@
     (property "Reference" "SW45" (id 0) (at 74.93 121.4882 0))
     (property "Value" "Rotary_Encoder_Switch" (id 1) (at 74.93 123.7996 0))
-    (property "Footprint" "Rotary_Encoder:RotaryEncoder_Alps_EC11E-Switch_Vertical_H20mm-SMD-support" (id 2) (at 71.12 126.746 0)
+    (property "Footprint" "Rotary_Encoder:RotaryEncoder_Alps_EC11E-Switch_Vertical_H20mm" (id 2) (at 71.12 126.746 0)
       (effects (font (size 1.27 1.27)) hide)
     )
@@
     (property "Reference" "NT1" (id 0) (at 27.94 62.23 0))
     (property "Value" "NetTie_2" (id 1) (at 27.94 65.0051 0))
-    (property "Footprint" "" (id 2) (at 27.94 63.5 0)
+    (property "Footprint" "NetTie:NetTie-2_SMD_Pad0.5mm" (id 2) (at 27.94 63.5 0)
       (effects (font (size 1.27 1.27)) hide)
     )
@@
     )
     (path "/db76666c-a33f-49b8-ae24-6f980f6cd506"
-      (reference "NT1") (unit 1) (value "NetTie_2") (footprint "")
+      (reference "NT1") (unit 1) (value "NetTie_2") (footprint "NetTie:NetTie-2_SMD_Pad0.5mm")
     )
     (path "/e05e05eb-3836-476f-a11a-aebc6024e210"
@@
     )
     (path "/cd2384f4-5ab3-4427-af04-4b5b6a978729"
-      (reference "SW45") (unit 1) (value "Rotary_Encoder_Switch") (footprint "Rotary_Encoder:RotaryEncoder_Alps_EC11E-Switch_Vertical_H20mm-SMD-support")
+      (reference "SW45") (unit 1) (value "Rotary_Encoder_Switch") (footprint "Rotary_Encoder:RotaryEncoder_Alps_EC11E-Switch_Vertical_H20mm")
     )
     (path "/253d01fc-0040-4948-ae39-949824a83cfa"

Commit message: PCB work started for RC-1
Parts:
- SW45: footprint Rotary_Encoder:RotaryEncoder_Alps_EC11E-Switch_Vertical_H20mm -> custom-encoders:EC11 THD&SMD
Connections:
- net col0: now also SW45_2.1; no longer SW45_2.2
- net at D45.2 (A), SW45.S2: now also SW45_2.2; no longer SW45_2.1
Other:
- moved on the sheet: SW45_2
Changed lines of the file:
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@@
   (junction (at 110.49 41.91) (diameter 0) (color 0 0 0 0)
   )
-  (junction (at 97.79 133.35) (diameter 0) (color 0 0 0 0)
-  )
   (junction (at 161.29 74.93) (diameter 0) (color 0 0 0 0)
   )
@@
   (junction (at 135.89 124.46) (diameter 0) (color 0 0 0 0)
   )
-  (junction (at 95.25 128.27) (diameter 0) (color 0 0 0 0)
-  )
   (junction (at 53.34 133.35) (diameter 0) (color 0 0 0 0)
   )
@@
   (junction (at 196.85 67.31) (diameter 0) (color 0 0 0 0)
   )
+  (junction (at 95.25 128.27) (diameter 0) (color 0 0 0 0)
+  )
   (junction (at 186.69 107.95) (diameter 0) (color 0 0 0 0)
   )
@@
   (junction (at 135.89 107.95) (diameter 0) (color 0 0 0 0)
   )
+  (junction (at 97.79 133.35) (diameter 0) (color 0 0 0 0)
+  )
   (junction (at 146.05 133.35) (diameter 0) (color 0 0 0 0)
   )
@@
     (stroke (width 0) (type default) (color 0 0 0 0))
   )
-  (wire (pts (xy 104.775 133.35) (xy 97.79 133.35))
+  (wire (pts (xy 82.55 133.35) (xy 97.79 133.35))
     (stroke (width 0) (type default) (color 0 0 0 0))
   )
@@
     (stroke (width 0) (type default) (color 0 0 0 0))
   )
+  (wire (pts (xy 107.95 128.27) (xy 107.95 132.715))
+    (stroke (width 0) (type default) (color 0 0 0 0))
+  )
   (wire (pts (xy 110.49 91.44) (xy 135.89 91.44))
     (stroke (width 0) (type default) (color 0 0 0 0))
@@
     (stroke (width 0) (type default) (color 0 0 0 0))
   )
-  (wire (pts (xy 104.775 136.525) (xy 104.775 133.35))
-    (stroke (width 0) (type default) (color 0 0 0 0))
-  )
   (wire (pts (xy 110.49 74.93) (xy 135.89 74.93))
     (stroke (width 0) (type default) (color 0 0 0 0))
@@
     (stroke (width 0) (type default) (color 0 0 0 0))
   )
-  (wire (pts (xy 95.25 128.27) (xy 104.775 128.27))
-    (stroke (width 0) (type default) (color 0 0 0 0))
-  )
   (wire (pts (xy 186.69 149.86) (xy 184.15 149.86))
     (stroke (width 0) (type default) (color 0 0 0 0))
@@
     (stroke (width 0) (type default) (color 0 0 0 0))
   )
-  (wire (pts (xy 114.935 128.27) (xy 114.935 136.525))
-    (stroke (width 0) (type default) (color 0 0 0 0))
-  )
   (wire (pts (xy 38.735 133.35) (xy 40.64 133.35))
     (stroke (width 0) (type default) (color 0 0 0 0))
@@
     (stroke (width 0) (type default) (color 0 0 0 0))
   )
+  (wire (pts (xy 118.11 132.715) (xy 118.11 136.525))
+    (stroke (width 0) (type default) (color 0 0 0 0))
+  )
   (wire (pts (xy 135.89 107.95) (xy 161.29 107.95))
     (stroke (width 0) (type default) (color 0 0 0 0))
@@
     (stroke (width 0) (type default) (color 0 0 0 0))
   )
-  (wire (pts (xy 224.79 67.31) (xy 222.25 67.31))
+  (wire (pts (xy 104.775 133.35) (xy 104.775 136.525))
     (stroke (width 0) (type default) (color 0 0 0 0))
   )
-  (wire (pts (xy 114.935 136.525) (xy 104.775 136.525))
+  (wire (pts (xy 224.79 67.31) (xy 222.25 67.31))
     (stroke (width 0) (type default) (color 0 0 0 0))
   )
@@
     (stroke (width 0) (type default) (color 0 0 0 0))
   )
-  (wire (pts (xy 95.25 128.27) (xy 95.25 149.86))
-    (stroke (width 0) (type default) (color 0 0 0 0))
-  )
   (wire (pts (xy 120.65 67.31) (xy 120.65 83.82))
     (stroke (width 0) (type default) (color 0 0 0 0))
@@
     (stroke (width 0) (type default) (color 0 0 0 0))
   )
-  (wire (pts (xy 82.55 133.35) (xy 97.79 133.35))
-    (stroke (width 0) (type default) (color 0 0 0 0))
-  )
   (wire (pts (xy 135.89 58.42) (xy 161.29 58.42))
     (stroke (width 0) (type default) (color 0 0 0 0))
@@
     (stroke (width 0) (type default) (color 0 0 0 0))
   )
+  (wire (pts (xy 97.79 133.35) (xy 104.775 133.35))
+    (stroke (width 0) (type default) (color 0 0 0 0))
+  )
   (wire (pts (xy 95.25 50.8) (xy 95.25 67.31))
     (stroke (width 0) (type default) (color 0 0 0 0))
@@
     (stroke (width 0) (type default) (color 0 0 0 0))
   )
+  (wire (pts (xy 82.55 128.27) (xy 95.25 128.27))
+    (stroke (width 0) (type default) (color 0 0 0 0))
+  )
   (wire (pts (xy 196.85 50.8) (xy 199.39 50.8))
     (stroke (width 0) (type default) (color 0 0 0 0))
@@
     (stroke (width 0) (type default) (color 0 0 0 0))
   )
-  (wire (pts (xy 82.55 128.27) (xy 95.25 128.27))
-    (stroke (width 0) (type default) (color 0 0 0 0))
-  )
   (wire (pts (xy 222.25 100.33) (xy 222.25 116.84))
     (stroke (width 0) (type default) (color 0 0 0 0))
@@
     (stroke (width 0) (type default) (color 0 0 0 0))
   )
+  (wire (pts (xy 95.25 128.27) (xy 107.95 128.27))
+    (stroke (width 0) (type default) (color 0 0 0 0))
+  )
   (wire (pts (xy 161.29 41.91) (xy 186.69 41.91))
     (stroke (width 0) (type default) (color 0 0 0 0))
@@
     (stroke (width 0) (type default) (color 0 0 0 0))
   )
+  (wire (pts (xy 118.11 136.525) (xy 104.775 136.525))
+    (stroke (width 0) (type default) (color 0 0 0 0))
+  )
+  (wire (pts (xy 95.25 128.27) (xy 95.25 149.86))
+    (stroke (width 0) (type default) (color 0 0 0 0))
+  )
   (wire (pts (xy 123.19 67.31) (xy 120.65 67.31))
     (stroke (width 0) (type default) (color 0 0 0 0))
@@
     (pin "1")
   )
-  (symbol (lib_id "Switch:SW_Push") (at 109.855 128.27 180) (unit 1)
+  (symbol (lib_id "Switch:SW_Push") (at 113.03 132.715 0) (unit 1)
     (in_bom yes) (on_board yes)
-    (property "Reference" "SW45_2" (id 0) (at 109.855 134.747 0))
-    (property "Value" "SW_PUSH" (id 1) (at 109.855 132.4356 0))
-    (property "Footprint" "keyswitches:SW_MX" (id 2) (at 109.855 128.27 0)
+    (property "Reference" "SW45_2" (id 0) (at 113.03 126.238 0))
+    (property "Value" "SW_PUSH" (id 1) (at 113.03 128.5494 0))
+    (property "Footprint" "keyswitches:SW_MX" (id 2) (at 113.03 132.715 0)
       (effects (font (size 1.27 1.27)) hide)
     )
-    (property "Datasheet" "" (id 3) (at 109.855 128.27 0))
+    (property "Datasheet" "" (id 3) (at 113.03 132.715 0))
     (pin "1")
     (pin "2")
@@
     (property "Reference" "SW45" (id 0) (at 74.93 121.4882 0))
     (property "Value" "Rotary_Encoder_Switch" (id 1) (at 74.93 123.7996 0))
-    (property "Footprint" "Rotary_Encoder:RotaryEncoder_Alps_EC11E-Switch_Vertical_H20mm" (id 2) (at 71.12 126.746 0)
+    (property "Footprint" "custom-encoders:EC11 THD&SMD" (id 2) (at 71.12 126.746 0)
       (effects (font (size 1.27 1.27)) hide)
     )
@@
     )
     (path "/cd2384f4-5ab3-4427-af04-4b5b6a978729"
-      (reference "SW45") (unit 1) (value "Rotary_Encoder_Switch") (footprint "Rotary_Encoder:RotaryEncoder_Alps_EC11E-Switch_Vertical_H20mm")
+      (reference "SW45") (unit 1) (value "Rotary_Encoder_Switch") (footprint "custom-encoders:EC11 THD&SMD")
     )
     (path "/253d01fc-0040-4948-ae39-949824a83cfa"

Commit message: todo: adjust component positions and reroute everything
Parts:
- C1, C2: footprint Capacitor_SMD:C_1206_3216Metric -> custom-electronics:Dual-Hybrid-1206-C_Disc_D4.3mm_W1.9mm_P5.00mm
Changed lines of the file:
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@@
       (effects (font (size 1.27 1.27)) (justify left))
     )
-    (property "Footprint" "Capacitor_SMD:C_1206_3216Metric" (id 2) (at 33.3502 140.97 0)
+    (property "Footprint" "custom-electronics:Dual-Hybrid-1206-C_Disc_D4.3mm_W1.9mm_P5.00mm" (id 2) (at 33.3502 140.97 0)
       (effects (font (size 1.27 1.27)) hide)
     )
@@
       (effects (font (size 1.27 1.27)) (justify left))
     )
-    (property "Footprint" "Capacitor_SMD:C_1206_3216Metric" (id 2) (at 33.3502 128.27 0)
+    (property "Footprint" "custom-electronics:Dual-Hybrid-1206-C_Disc_D4.3mm_W1.9mm_P5.00mm" (id 2) (at 33.3502 128.27 0)
       (effects (font (size 1.27 1.27)) hide)
     )
@@
     )
     (path "/a75a6b6e-fd3e-4beb-a876-b0db64cea578"
-      (reference "C1") (unit 1) (value "C") (footprint "Capacitor_SMD:C_1206_3216Metric")
+      (reference "C1") (unit 1) (value "C") (footprint "custom-electronics:Dual-Hybrid-1206-C_Disc_D4.3mm_W1.9mm_P5.00mm")
     )
     (path "/d44f6aaa-f8db-4ae4-8055-30867637d971"
-      (reference "C2") (unit 1) (value "C") (footprint "Capacitor_SMD:C_1206_3216Metric")
+      (reference "C2") (unit 1) (value "C") (footprint "custom-electronics:Dual-Hybrid-1206-C_Disc_D4.3mm_W1.9mm_P5.00mm")
     )
     (path "/00000000-0000-0000-0000-00005dcbd469"

Commit message: revise ver1.0 RC-1 routing; remove redudant backups
Parts:
- removed NT1: NetTie_2, NetTie:NetTie-2_SMD_Pad0.5mm, symbol Device:NetTie_2
- U1: footprint promicro-nicenano:promicro-nicenano -> Keebio-Parts:ArduinoProMicro; symbol promicro-nicenano:promicro-nicenano -> promicro:ProMicro
Connections:
- net GND: now also SW_PWR1.3, U1.23 (GND); no longer U1.14 (GND)
- net VCC: now also U1.21 (VCC); no longer U1.16 (VCC)
- net reset: now also U1.22 (RST); no longer U1.15 (RST)
- net row0: now also U1.20 (F4); no longer U1.17 (F4)
- net row1: now also U1.19 (F5); no longer U1.18 (F5)
- net row2: now also U1.18 (F6); no longer U1.19 (F6)
- net row3: now also U1.17 (F7); no longer U1.20 (F7)
- net row4: now also U1.16 (B1); no longer U1.21 (B1)
- net row5: now also U1.15 (B3); no longer U1.22 (B3)
- net row6: now also U1.14 (B2); no longer U1.23 (B2)
- net at U1.24 (RAW): now also SW_PWR1.1
- no-connect marks 3 -> 2
Changed lines of the file:
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@@
   (junction (at 95.25 67.31) (diameter 0) (color 0 0 0 0)
   )
-  (junction (at 32.385 63.5) (diameter 0) (color 0 0 0 0)
-  )
   (junction (at 110.49 74.93) (diameter 0) (color 0 0 0 0)
   )
@@
   (no_connect (at 32.385 66.04))
   (no_connect (at 67.945 93.98))
-  (no_connect (at 67.945 66.04))
   (wire (pts (xy 85.09 179.07) (xy 85.09 181.61))
     (stroke (width 0) (type default) (color 0 0 0 0))
   )
-  (wire (pts (xy 32.385 52.07) (xy 32.385 63.5))
-    (stroke (width 0) (type default) (color 0 0 0 0))
-  )
   (wire (pts (xy 146.05 83.82) (xy 148.59 83.82))
     (stroke (width 0) (type default) (color 0 0 0 0))
@@
     (stroke (width 0) (type default) (color 0 0 0 0))
   )
+  (wire (pts (xy 46.99 49.53) (xy 46.99 52.07))
+    (stroke (width 0) (type default) (color 0 0 0 0))
+  )
   (wire (pts (xy 186.69 133.35) (xy 184.15 133.35))
     (stroke (width 0) (type default) (color 0 0 0 0))
@@
     (stroke (width 0) (type default) (color 0 0 0 0))
   )
+  (wire (pts (xy 69.85 66.04) (xy 67.945 66.04))
+    (stroke (width 0) (type default) (color 0 0 0 0))
+  )
   (wire (pts (xy 146.05 83.82) (xy 146.05 100.33))
     (stroke (width 0) (type default) (color 0 0 0 0))
@@
     (stroke (width 0) (type default) (color 0 0 0 0))
   )
-  (wire (pts (xy 46.99 49.53) (xy 46.99 52.07))
-    (stroke (width 0) (type default) (color 0 0 0 0))
-  )
   (wire (pts (xy 120.65 50.8) (xy 123.19 50.8))
     (stroke (width 0) (type default) (color 0 0 0 0))
@@
     (stroke (width 0) (type default) (color 0 0 0 0))
   )
-  (wire (pts (xy 24.13 63.5) (xy 25.4 63.5))
-    (stroke (width 0) (type default) (color 0 0 0 0))
-  )
   (wire (pts (xy 184.15 116.84) (xy 186.69 116.84))
     (stroke (width 0) (type default) (color 0 0 0 0))
@@
     (stroke (width 0) (type default) (color 0 0 0 0))
   )
+  (wire (pts (xy 46.99 52.07) (xy 31.115 52.07))
+    (stroke (width 0) (type default) (color 0 0 0 0))
+  )
   (wire (pts (xy 135.89 107.95) (xy 161.29 107.95))
     (stroke (width 0) (type default) (color 0 0 0 0))
@@
     (stroke (width 0) (type default) (color 0 0 0 0))
   )
+  (wire (pts (xy 69.85 52.07) (xy 69.85 66.04))
+    (stroke (width 0) (type default) (color 0 0 0 0))
+  )
   (wire (pts (xy 196.85 34.29) (xy 196.85 50.8))
     (stroke (width 0) (type default) (color 0 0 0 0))
@@
     (stroke (width 0) (type default) (color 0 0 0 0))
   )
-  (wire (pts (xy 30.48 63.5) (xy 32.385 63.5))
-    (stroke (width 0) (type default) (color 0 0 0 0))
-  )
   (wire (pts (xy 196.85 67.31) (xy 196.85 83.82))
     (stroke (width 0) (type default) (color 0 0 0 0))
@@
     (stroke (width 0) (type default) (color 0 0 0 0))
   )
-  (wire (pts (xy 46.99 52.07) (xy 32.385 52.07))
-    (stroke (width 0) (type default) (color 0 0 0 0))
-  )
   (wire (pts (xy 38.735 118.11) (xy 38.735 128.27))
     (stroke (width 0) (type default) (color 0 0 0 0))
@@
     (stroke (width 0) (type default) (color 0 0 0 0))
   )
-  (wire (pts (xy 67.945 63.5) (xy 67.945 52.07))
-    (stroke (width 0) (type default) (color 0 0 0 0))
-  )
   (wire (pts (xy 158.75 83.82) (xy 161.29 83.82))
     (stroke (width 0) (type default) (color 0 0 0 0))
@@
     (stroke (width 0) (type default) (color 0 0 0 0))
   )
-  (wire (pts (xy 67.945 52.07) (xy 52.07 52.07))
+  (wire (pts (xy 52.07 52.07) (xy 69.85 52.07))
     (stroke (width 0) (type default) (color 0 0 0 0))
   )
@@
     (pin "1")
   )
-  (symbol (lib_id "promicro-nicenano:promicro-nicenano") (at 50.165 85.09 0) (unit 1)
+  (symbol (lib_id "promicro:ProMicro") (at 50.165 85.09 0) (unit 1)
     (in_bom yes) (on_board yes)
     (property "Reference" "U1" (id 0) (at 50.165 54.9402 0)
@@
       (effects (font (size 1.524 1.524)))
     )
-    (property "Footprint" "promicro-nicenano:promicro-nicenano" (id 2) (at 50.165 102.235 0)
+    (property "Footprint" "Keebio-Parts:ArduinoProMicro" (id 2) (at 52.705 111.76 0)
       (effects (font (size 1.524 1.524)))
     )
@@
     (pin "23")
     (pin "24")
-    (pin "25")
-    (pin "26")
     (pin "3")
     (pin "4")
@@
     (pin "2")
   )
-  (symbol (lib_id "power:GND") (at 24.13 63.5 270) (unit 1)
+  (symbol (lib_id "power:GND") (at 31.115 52.07 270) (unit 1)
     (in_bom yes) (on_board yes)
-    (property "Reference" "#PWR0104" (id 0) (at 17.78 63.5 0)
+    (property "Reference" "#PWR0104" (id 0) (at 24.765 52.07 0)
       (effects (font (size 1.27 1.27)) hide)
     )
-    (property "Value" "GND" (id 1) (at 20.8788 63.627 90)
+    (property "Value" "GND" (id 1) (at 27.8638 52.197 90)
       (effects (font (size 1.27 1.27)) (justify right))
     )
-    (property "Footprint" "" (id 2) (at 24.13 63.5 0)
+    (property "Footprint" "" (id 2) (at 31.115 52.07 0)
       (effects (font (size 1.27 1.27)) hide)
     )
-    (property "Datasheet" "" (id 3) (at 24.13 63.5 0)
+    (property "Datasheet" "" (id 3) (at 31.115 52.07 0)
       (effects (font (size 1.27 1.27)) hide)
     )
@@
     (pin "2")
   )
-  (symbol (lib_id "Device:NetTie_2") (at 27.94 63.5 0) (unit 1)
-    (in_bom yes) (on_board yes)
-    (property "Reference" "NT1" (id 0) (at 27.94 62.23 0))
-    (property "Value" "NetTie_2" (id 1) (at 27.94 65.0051 0))
-    (property "Footprint" "NetTie:NetTie-2_SMD_Pad0.5mm" (id 2) (at 27.94 63.5 0)
-      (effects (font (size 1.27 1.27)) hide)
-    )
-    (property "Datasheet" "~" (id 3) (at 27.94 63.5 0)
-      (effects (font (size 1.27 1.27)) hide)
-    )
-    (pin "1")
-    (pin "2")
-  )
   (symbol (lib_id "Device:R") (at 44.45 133.35 90) (unit 1)
     (in_bom yes) (on_board yes)
@@
       (reference "JP2") (unit 1) (value "SolderJumper_2_Open") (footprint "Jumper:SolderJumper-2_P1.3mm_Open_Pad1.0x1.5mm")
     )
-    (path "/db76666c-a33f-49b8-ae24-6f980f6cd506"
-      (reference "NT1") (unit 1) (value "NetTie_2") (footprint "NetTie:NetTie-2_SMD_Pad0.5mm")
-    )
     (path "/e05e05eb-3836-476f-a11a-aebc6024e210"
       (reference "R1") (unit 1) (value "R") (footprint "Resistor_THT:R_Axial_DIN0204_L3.6mm_D1.6mm_P7.62mm_Horizontal")
@@
     )
     (path "/00000000-0000-0000-0000-00005dcbb133"
-      (reference "U1") (unit 1) (value "ProMicro/Nice!Nano") (footprint "promicro-nicenano:promicro-nicenano")
+      (reference "U1") (unit 1) (value "ProMicro/Nice!Nano") (footprint "Keebio-Parts:ArduinoProMicro")
     )
   )

Commit message: WIP: major layout reworks
Parts:
- removed SW45_2: SW_PUSH, keyswitches:SW_MX, symbol Switch:SW_Push
- BT1: footprint Connector_PinHeader_2.00mm:PinHeader_1x02_P2.00mm_Vertical -> Connector_JST:JST_PH_S2B-PH-K_1x02_P2.00mm_Horizontal
- SW45: footprint custom-encoders:EC11 THD&SMD -> custom-encoders:EC11_THD_SMD_With_Switch
Connections:
- net row3: now also D37.1 (K), D38.1 (K), D39.1 (K), D40.1 (K), D45.1 (K); no longer D19.1 (K), D20.1 (K), D21.1 (K), D22.1 (K), D23.1 (K), D24.1 (K)
- net row4: now also D19.1 (K), D20.1 (K), D21.1 (K), D22.1 (K), D23.1 (K), D24.1 (K), U1.13 (B6); no longer D25.1 (K), D26.1 (K), D27.1 (K), D28.1 (K), D29.1 (K), D30.1 (K), U1.16 (B1)
- net row5: now also D25.1 (K), D26.1 (K), D27.1 (K), D28.1 (K), D29.1 (K), D30.1 (K), U1.14 (B2); no longer D31.1 (K), D32.1 (K), D33.1 (K), D34.1 (K), D35.1 (K), D36.1 (K), U1.15 (B3)
- net row6: now also D31.1 (K), D32.1 (K), D33.1 (K), D34.1 (K), D35.1 (K), D36.1 (K), U1.15 (B3); no longer D37.1 (K), D38.1 (K), D39.1 (K), D40.1 (K), D45.1 (K), U1.14 (B2)
- net row7: now also U1.16 (B1); no longer U1.2 (RX)
Other:
- moved on the sheet: BT1, C1, C2, D1, D10, D11, D12, D13, D14, D15, D16, D17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

Commit message: Change to Single Sided SMD diodes; continue trace rework
Parts:
- D1, D10, D11, D12, D13, D14, D15, D16, D17, D18, D19, D2, D20, D21, D22, D23, D24, D25, D26, D27, D28, D29, D3, D30, D31, D32, D33, D34, D35, D36, D37, D38, D39, D4, D40, D41, D42, D43, D44, D45, D5, D6, D7, D8, D9: footprint Keebio-Parts:Diode-dual -> Keebio-Parts:Diode-Hybrid-Back
