File: kicad/ver1.0 RC-1/pcb/choctopus44.kicad_sch (KiCad schematic)
At the start: 102 parts, among them SW1 SW_PUSH, SW10 SW_PUSH, SW11 SW_PUSH, SW12 SW_PUSH, SW13 SW_PUSH, SW14 SW_PUSH, SW15 SW_PUSH, SW16 SW_PUSH, SW17 SW_PUSH, SW18 SW_PUSH, SW19 SW_PUSH, SW2 SW_PUSH, SW20 SW_PUSH, SW21 SW_PUSH, SW22 SW_PUSH, SW23 SW_PUSH, SW24 SW_PUSH, SW25 SW_PUSH, SW26 SW_PUSH, SW27 SW_PUSH, SW28 SW_PUSH, SW29 SW_PUSH, SW3 SW_PUSH, SW30 SW_PUSH, SW31 SW_PUSH, SW32 SW_PUSH, SW33 SW_PUSH, SW34 SW_PUSH, SW35 SW_PUSH, SW36 SW_PUSH, SW37 SW_PUSH, SW38 SW_PUSH, SW39 SW_PUSH, SW4 SW_PUSH, SW40 SW_PUSH, SW41 SW_PUSH, SW42 SW_PUSH, SW43 SW_PUSH, SW44 SW_PUSH, SW45 Rotary_Encoder_Switch, SW5 SW_PUSH, SW6 SW_PUSH, SW7 SW_PUSH, SW8 SW_PUSH, SW9 SW_PUSH, U1 ProMicro/Nice!Nano

Commit message: initial error-free routing for RC-1
Parts:
- BT1: footprint Connector_JST:JST_PH_S2B-PH-K_1x02_P2.00mm_Horizontal -> Connector_PinHeader_2.00mm:PinHeader_1x02_P2.00mm_Vertical
- RESET1: symbol Switch:SW_DPST -> Switch:SW_MEC_5E
- SW45: footprint custom-encoders:EC11_THD_SMD_With_Switch -> custom-encoders:EC11_THD_SMD_Choc_MX
Connections:
- net GND: now also RESET1.3 (K), SW_PWR1.2; no longer RESET1.2, SW_PWR1.3
- net reset: now also RESET1.2; no longer RESET1.3
- net at U1.24 (RAW): now also SW_PWR1.4; no longer SW_PWR1.1
- net at BT1.1 (+): now also SW_PWR1.3; no longer SW_PWR1.2
- net at BT1.2 (-): now also SW_PWR1.1; no longer SW_PWR1.4
Other:
- moved on the sheet: SW_PWR1
Changed lines of the file:
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@@
   (junction (at 163.195 115.57) (diameter 0) (color 0 0 0 0)
   )
+  (junction (at 60.96 50.8) (diameter 0) (color 0 0 0 0)
+  )
   (junction (at 178.435 89.535) (diameter 0) (color 0 0 0 0)
   )
@@
   (junction (at 163.195 48.895) (diameter 0) (color 0 0 0 0)
   )
+  (junction (at 50.8 50.8) (diameter 0) (color 0 0 0 0)
+  )
   (junction (at 188.595 65.405) (diameter 0) (color 0 0 0 0)
   )
@@
   (junction (at 64.77 76.835) (diameter 0) (color 0 0 0 0)
   )
-  (junction (at 50.8 46.355) (diameter 0) (color 0 0 0 0)
-  )
-  (junction (at 60.96 46.355) (diameter 0) (color 0 0 0 0)
-  )
   (junction (at 178.435 106.68) (diameter 0) (color 0 0 0 0)
   )
@@
   (no_connect (at 42.545 151.765))
   (no_connect (at 42.545 154.305))
-  (wire (pts (xy 50.8 46.355) (xy 50.8 48.895))
-    (stroke (width 0) (type default) (color 0 0 0 0))
-  )
   (wire (pts (xy 163.195 99.06) (xy 165.735 99.06))
     (stroke (width 0) (type default) (color 0 0 0 0))
@@
     (stroke (width 0) (type default) (color 0 0 0 0))
   )
+  (wire (pts (xy 60.96 50.8) (xy 64.77 50.8))
+    (stroke (width 0) (type default) (color 0 0 0 0))
+  )
   (wire (pts (xy 203.835 123.19) (xy 229.235 123.19))
     (stroke (width 0) (type default) (color 0 0 0 0))
@@
     (stroke (width 0) (type default) (color 0 0 0 0))
   )
-  (wire (pts (xy 60.96 48.895) (xy 60.96 46.355))
-    (stroke (width 0) (type default) (color 0 0 0 0))
-  )
   (wire (pts (xy 137.795 149.225) (xy 140.335 149.225))
     (stroke (width 0) (type default) (color 0 0 0 0))
@@
     (stroke (width 0) (type default) (color 0 0 0 0))
   )
-  (wire (pts (xy 60.96 43.815) (xy 60.96 46.355))
-    (stroke (width 0) (type default) (color 0 0 0 0))
-  )
   (wire (pts (xy 81.28 76.835) (xy 81.915 76.835))
     (stroke (width 0) (type default) (color 0 0 0 0))
@@
     (stroke (width 0) (type default) (color 0 0 0 0))
   )
-  (wire (pts (xy 50.8 46.355) (xy 50.8 43.815))
-    (stroke (width 0) (type default) (color 0 0 0 0))
-  )
   (wire (pts (xy 203.835 73.025) (xy 229.235 73.025))
     (stroke (width 0) (type default) (color 0 0 0 0))
@@
     (stroke (width 0) (type default) (color 0 0 0 0))
   )
+  (wire (pts (xy 50.8 50.8) (xy 50.8 52.07))
+    (stroke (width 0) (type default) (color 0 0 0 0))
+  )
   (wire (pts (xy 203.835 81.915) (xy 201.295 81.915))
     (stroke (width 0) (type default) (color 0 0 0 0))
@@
     (stroke (width 0) (type default) (color 0 0 0 0))
   )
+  (wire (pts (xy 50.8 49.53) (xy 50.8 50.8))
+    (stroke (width 0) (type default) (color 0 0 0 0))
+  )
   (wire (pts (xy 254.635 65.405) (xy 252.095 65.405))
     (stroke (width 0) (type default) (color 0 0 0 0))
@@
     (stroke (width 0) (type default) (color 0 0 0 0))
   )
-  (wire (pts (xy 60.96 46.355) (xy 63.5 46.355))
-    (stroke (width 0) (type default) (color 0 0 0 0))
-  )
   (wire (pts (xy 71.12 76.835) (xy 81.28 76.835))
     (stroke (width 0) (type default) (color 0 0 0 0))
@@
     (stroke (width 0) (type default) (color 0 0 0 0))
   )
+  (wire (pts (xy 46.99 50.8) (xy 50.8 50.8))
+    (stroke (width 0) (type default) (color 0 0 0 0))
+  )
   (wire (pts (xy 239.395 65.405) (xy 239.395 81.915))
     (stroke (width 0) (type default) (color 0 0 0 0))
@@
     (stroke (width 0) (type default) (color 0 0 0 0))
   )
+  (wire (pts (xy 60.96 50.8) (xy 60.96 52.07))
+    (stroke (width 0) (type default) (color 0 0 0 0))
+  )
   (wire (pts (xy 239.395 24.765) (xy 239.395 32.385))
     (stroke (width 0) (type default) (color 0 0 0 0))
@@
     (stroke (width 0) (type default) (color 0 0 0 0))
   )
+  (wire (pts (xy 60.96 49.53) (xy 60.96 50.8))
+    (stroke (width 0) (type default) (color 0 0 0 0))
+  )
   (wire (pts (xy 239.395 99.06) (xy 241.935 99.06))
     (stroke (width 0) (type default) (color 0 0 0 0))
@@
     (stroke (width 0) (type default) (color 0 0 0 0))
   )
-  (wire (pts (xy 48.26 46.355) (xy 50.8 46.355))
-    (stroke (width 0) (type default) (color 0 0 0 0))
-  )
   (wire (pts (xy 175.895 32.385) (xy 178.435 32.385))
     (stroke (width 0) (type default) (color 0 0 0 0))
@@
     )
   )
-  (global_label "reset" (shape input) (at 48.26 46.355 180) (fields_autoplaced)
+  (global_label "reset" (shape input) (at 46.99 50.8 180) (fields_autoplaced)
     (effects (font (size 1.27 1.27)) (justify right))
-    (property "Intersheet References" "${INTERSHEET_REFS}" (id 0) (at -34.29 -132.715 0)
+    (property "Intersheet References" "${INTERSHEET_REFS}" (id 0) (at -35.56 -128.27 0)
       (effects (font (size 1.27 1.27)) hide)
     )
@@
     (pin "2")
   )
-  (symbol (lib_id "Switch:SW_DPST") (at 55.88 46.355 0) (unit 1)
+  (symbol (lib_id "Switch:SW_MEC_5E") (at 55.88 52.07 0) (unit 1)
     (in_bom yes) (on_board yes)
-    (property "Reference" "RESET1" (id 0) (at 55.88 39.878 0))
-    (property "Value" "SW_PUSH" (id 1) (at 55.88 42.1894 0))
-    (property "Footprint" "Button_Switch_THT:SW_TH_Tactile_Omron_B3F-10xx" (id 2) (at 55.88 46.355 0)
+    (property "Reference" "RESET1" (id 0) (at 55.88 43.18 0))
+    (property "Value" "SW_PUSH" (id 1) (at 55.88 45.4914 0))
+    (property "Footprint" "Button_Switch_THT:SW_TH_Tactile_Omron_B3F-10xx" (id 2) (at 55.88 44.45 0)
+      (effects (font (size 1.27 1.27)) hide)
+    )
+    (property "Datasheet" "http://www.apem.com/int/index.php?controller=attachment&id_attachment=1371" (id 3) (at 55.88 44.45 0)
       (effects (font (size 1.27 1.27)) hide)
     )
-    (property "Datasheet" "" (id 3) (at 55.88 46.355 0))
     (pin "1")
     (pin "2")
@@
     (pin "4")
   )
-  (symbol (lib_id "power:GND") (at 63.5 46.355 90) (unit 1)
+  (symbol (lib_id "power:GND") (at 64.77 50.8 90) (unit 1)
     (in_bom yes) (on_board yes)
-    (property "Reference" "#PWR08" (id 0) (at 69.85 46.355 0)
+    (property "Reference" "#PWR08" (id 0) (at 71.12 50.8 0)
       (effects (font (size 1.27 1.27)) hide)
     )
-    (property "Value" "GND" (id 1) (at 66.7512 46.228 90)
+    (property "Value" "GND" (id 1) (at 67.945 50.8 90)
       (effects (font (size 1.27 1.27)) (justify right))
     )
-    (property "Footprint" "" (id 2) (at 63.5 46.355 0)
+    (property "Footprint" "" (id 2) (at 64.77 50.8 0)
       (effects (font (size 1.27 1.27)) hide)
     )
-    (property "Datasheet" "" (id 3) (at 63.5 46.355 0)
+    (property "Datasheet" "" (id 3) (at 64.77 50.8 0)
       (effects (font (size 1.27 1.27)) hide)
     )
@@
     (pin "2")
   )
-  (symbol (lib_id "Switch:SW_DPST") (at 59.69 130.175 90) (unit 1)
+  (symbol (lib_id "Switch:SW_DPST") (at 59.69 130.175 270) (unit 1)
     (in_bom yes) (on_board yes)
-    (property "Reference" "SW_PWR1" (id 0) (at 51.435 130.175 0))
-    (property "Value" "SW_DPST" (id 1) (at 53.7464 130.175 0))
+    (property "Reference" "SW_PWR1" (id 0) (at 67.945 130.175 0))
+    (property "Value" "SW_DPST" (id 1) (at 65.6336 130.175 0))
     (property "Footprint" "Button_Switch_THT:SW_E-Switch_EG1271_DPDT" (id 2) (at 59.69 130.175 0)
       (effects (font (size 1.27 1.27)) hide)
@@
       (effects (font (size 1.27 1.27)) (justify left))
     )
-    (property "Footprint" "Connector_JST:JST_PH_S2B-PH-K_1x02_P2.00mm_Horizontal" (id 2) (at 59.944 116.205 90)
+    (property "Footprint" "Connector_PinHeader_2.00mm:PinHeader_1x02_P2.00mm_Vertical" (id 2) (at 59.944 116.205 90)
       (effects (font (size 1.27 1.27)) hide)
     )
@@
     (property "Reference" "SW45" (id 0) (at 88.9 70.0532 0))
     (property "Value" "Rotary_Encoder_Switch" (id 1) (at 88.9 72.3646 0))
-    (property "Footprint" "custom-encoders:EC11_THD_SMD_With_Switch" (id 2) (at 85.09 75.311 0)
+    (property "Footprint" "custom-encoders:EC11_THD_SMD_Choc_MX" (id 2) (at 85.09 75.311 0)
       (effects (font (size 1.27 1.27)) hide)
     )
@@
     )
     (path "/00000000-0000-0000-0000-000060df8fe8"
-      (reference "BT1") (unit 1) (value "Battery_Cell") (footprint "Connector_JST:JST_PH_S2B-PH-K_1x02_P2.00mm_Horizontal")
+      (reference "BT1") (unit 1) (value "Battery_Cell") (footprint "Connector_PinHeader_2.00mm:PinHeader_1x02_P2.00mm_Vertical")
     )
     (path "/a75a6b6e-fd3e-4beb-a876-b0db64cea578"
@@
     )
     (path "/cd2384f4-5ab3-4427-af04-4b5b6a978729"
-      (reference "SW45") (unit 1) (value "Rotary_Encoder_Switch") (footprint "custom-encoders:EC11_THD_SMD_With_Switch")
+      (reference "SW45") (unit 1) (value "Rotary_Encoder_Switch") (footprint "custom-encoders:EC11_THD_SMD_Choc_MX")
     )
     (path "/00000000-0000-0000-0000-000060df3383"
