File: kicad/ver2.0/pcb-top-plate/choctopus44-top-plate.kicad_pcb (KiCad board)
At the start: 2 copper layers, 243.9 x 119.3 mm, 78 parts, among them SW1 SW_PUSH, SW10 SW_PUSH, SW11 SW_PUSH, SW12 SW_PUSH, SW13 SW_PUSH, SW14 SW_PUSH, SW15 SW_PUSH, SW16 SW_PUSH, SW17 SW_PUSH, SW18 SW_PUSH, SW19 SW_PUSH, SW2 SW_PUSH, SW20 SW_PUSH, SW21 SW_PUSH, SW22 SW_PUSH, SW23 SW_PUSH, SW24 SW_PUSH, SW25 SW_PUSH, SW26 SW_PUSH, SW27 SW_PUSH, SW28 SW_PUSH, SW29 SW_PUSH, SW3 SW_PUSH, SW30 SW_PUSH, SW31 SW_PUSH, SW32 SW_PUSH, SW33 SW_PUSH, SW34 SW_PUSH, SW35 SW_PUSH, SW36 SW_PUSH, SW37 SW_PUSH, SW38 SW_PUSH, SW39 SW_PUSH, SW4 SW_PUSH, SW40 SW_PUSH, SW41 SW_PUSH, SW42 SW_PUSH, SW43 SW_PUSH, SW44 SW_PUSH, SW5 SW_PUSH, SW6 SW_PUSH, SW7 SW_PUSH, SW8 SW_PUSH, SW9 SW_PUSH

Commit message: initial switch plate files
Parts:
- removed G***: LOGO, keyboard stuff:routa-logo-smallish
- removed H12 (x2): H12, MountingHole:MountingHole_2.2mm_M2
- removed H13 (x2): H13, MountingHole:MountingHole_2.2mm_M2
- removed H14: H14, MountingHole:MountingHole_2.2mm_M2
- removed the H6 at (144.7, 109.7)
- removed the H6 at (142.5, 106.0)
- removed the H6 at (149.0, 109.7)
- removed the H6 at (144.7, 102.2)
- removed the H6 at (146.8, 98.5)
- removed the H6 at (144.7, 94.8)
- removed the H6 at (140.4, 102.2)
- removed the H6 at (146.8, 113.4)
- removed the H6 at (149.0, 102.2)
- removed the H6 at (142.5, 98.5)
- removed the H6 at (146.8, 91.1)
- removed the H6 at (151.1, 113.4)
- removed the H6 at (140.4, 109.7)
- removed the H6 at (146.8, 106.0)
- removed the H6 at (144.7, 154.5)
- removed the H6 at (138.2, 113.4)
- removed the H6 at (149.0, 117.1)
- removed the H6 at (140.4, 117.1)
- removed the H6 at (144.7, 117.1)
- removed the H6 at (144.7, 87.3)
- removed the H6 at (142.5, 91.1)
- removed the H6 at (142.5, 113.4)
- removed the H8 at (89.6, 111.2)
- removed the H8 at (199.8, 111.2)
- removed mouse-bite-2mm-slot (x2): VAL**, Panelization:mouse-bite-4-25-x-3-slot
- added H6: H6, MountingHole:MountingHole_2.2mm_M2_ISO14580_Pad, F.Cu at (148.3, 156.7)
- added H6: H6, MountingHole:MountingHole_2.2mm_M2_ISO14580_Pad, F.Cu at (147.7, 48.6)
- added H6: H6, MountingHole:MountingHole_2.2mm_M2_ISO14580_Pad, F.Cu at (159.8, 58.0)
- added H6: H6, MountingHole:MountingHole_2.2mm_M2_ISO14580_Pad, F.Cu at (135.9, 74.4)
- added H6: H6, MountingHole:MountingHole_2.2mm_M2_ISO14580_Pad, F.Cu at (123.5, 49.8)
- added H6: H6, MountingHole:MountingHole_2.2mm_M2_ISO14580_Pad, F.Cu at (123.8, 65.0)
- added H6: H6, MountingHole:MountingHole_2.2mm_M2_ISO14580_Pad, F.Cu at (160.1, 73.2)
- added H6: H6, MountingHole:MountingHole_2.2mm_M2_ISO14580_Pad, F.Cu at (148.3, 111.9)
- added H8: H8, MountingHole:MountingHole_2.2mm_M2_ISO14580_Pad, F.Cu at (225.0, 109.4)
- added H8: H8, MountingHole:MountingHole_2.2mm_M2_ISO14580_Pad, B.Cu at (71.5, 109.4)
- added REF**: breakaway-mousebites, Keebio-Parts:breakaway-mousebites, F.Cu at (143.9, 73.5)
- added REF**: breakaway-mousebites, Keebio-Parts:breakaway-mousebites, F.Cu at (130.0, 65.4)
- added REF**: breakaway-mousebites, Keebio-Parts:breakaway-mousebites, F.Cu at (142.1, 75.6)
- added REF**: breakaway-mousebites, Keebio-Parts:breakaway-mousebites, F.Cu at (131.7, 63.4)
- added SW45: Rotary_Encoder_Switch, custom-electronics:custom-ec11-cutout, F.Cu at (148.3, 131.7)
- H1: value MountingHole -> H1
- SW1, SW10, SW11, SW12, SW13, SW14, SW15, SW16, SW17, SW18, SW19, SW2, SW20, SW21, SW22, SW23, SW24, SW25, SW26, SW27, SW28, SW29, SW3, SW30, SW31, SW32, SW33, SW34, SW35, SW36, SW37, SW38, SW39, SW4, SW40, SW41, SW42, SW43, SW44, SW5, SW6, SW7, SW8, SW9: footprint Keyboard:MXPLATE-1U -> custom-electronics:choc-plate-cutout
- moved SW36 8.54 mm to (257.8, 94.2), turned to 20 degrees
- moved H1 8.02 mm to (75.6, 58.5), turned to -5 degrees
- moved SW1 7.97 mm to (50.3, 62.2), turned to -20 degrees
- moved SW35 7.71 mm to (240.9, 100.3), turned to 20 degrees
- moved SW7 7.55 mm to (44.5, 78.2), turned to -20 degrees
- moved SW13 7.44 mm to (38.7, 94.2), turned to -20 degrees
- moved SW30 7.38 mm to (252.0, 78.2), turned to 20 degrees
- moved SW31 6.85 mm to (171.3, 119.7), turned to 20 degrees
- moved SW2 6.58 mm to (67.2, 68.4), turned to -20 degrees
- moved SW29 6.40 mm to (235.1, 84.4), turned to 20 degrees
- moved SW24 6.38 mm to (246.2, 62.2), turned to 20 degrees
- moved SW34 6.21 mm to (220.8, 97.8), turned to 20 degrees
- moved SW41 6.15 mm to (162.4, 151.4), turned to 45 degrees
- moved SW32 6.09 mm to (187.0, 110.1), turned to 20 degrees
- moved SW8 6.07 mm to (61.4, 84.4), turned to -20 degrees
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Other:
- board size 243.9 x 119.3 mm -> 247.4 x 124.8 mm
- net class Default removed
- board text added: "4.5; 2.75"
- board text added: "Choctopus44v2 by Routa Keebs 2023 Loosely based on Reviung41 rev1.3 GH by gtips 2021"
- board text removed: "CHOCTOPUS44"
- board text removed: "Choctopus44 [Prototype]"
- board text removed: "Choctopus44 [Prototype] By Routa#1858/SlightHeadache"
