File: kicad/ver2.0/pcb-top-plate/choctopus44-top-plate.kicad_pcb (KiCad board)
At the start: 2 copper layers, 247.4 x 124.8 mm, 61 parts, among them SW1 SW_PUSH, SW10 SW_PUSH, SW11 SW_PUSH, SW12 SW_PUSH, SW13 SW_PUSH, SW14 SW_PUSH, SW15 SW_PUSH, SW16 SW_PUSH, SW17 SW_PUSH, SW18 SW_PUSH, SW19 SW_PUSH, SW2 SW_PUSH, SW20 SW_PUSH, SW21 SW_PUSH, SW22 SW_PUSH, SW23 SW_PUSH, SW24 SW_PUSH, SW25 SW_PUSH, SW26 SW_PUSH, SW27 SW_PUSH, SW28 SW_PUSH, SW29 SW_PUSH, SW3 SW_PUSH, SW30 SW_PUSH, SW31 SW_PUSH, SW32 SW_PUSH, SW33 SW_PUSH, SW34 SW_PUSH, SW35 SW_PUSH, SW36 SW_PUSH, SW37 SW_PUSH, SW38 SW_PUSH, SW39 SW_PUSH, SW4 SW_PUSH, SW40 SW_PUSH, SW41 SW_PUSH, SW42 SW_PUSH, SW43 SW_PUSH, SW44 SW_PUSH, SW45 Rotary_Encoder_Switch, SW5 SW_PUSH, SW6 SW_PUSH, SW7 SW_PUSH, SW8 SW_PUSH, SW9 SW_PUSH

Commit message: silk screen changes
Parts:
- added G***: LOGO, keyboard stuff:mustekala-2-17mm, F.Cu at (148.3, 102.9)
- added G***: LOGO, keyboard stuff:routa-logo-smaller, B.Cu at (157.4, 118.7)
- moved H6 3.72 mm to (121.5, 46.7)
- moved H6 3.72 mm to (145.7, 45.5)
- moved H6 3.72 mm to (157.7, 54.9)
- moved REF** 3.72 mm to (129.7, 60.3)
- moved REF** 3.72 mm to (141.8, 70.4)
- moved REF** 3.60 mm to (127.3, 63.1)
- moved REF** 3.60 mm to (139.4, 73.3)
Other:
- board size 247.4 x 124.8 mm -> 247.4 x 127.9 mm
- board text added: "Choctopus44v2"

Commit message: new gerbers etc
Parts:
- added G***: LOGO, keyboard stuff:choctopus-logo-3-40mm, F.Cu at (140.2, 55.2)
- G***: footprint keyboard stuff:mustekala-2-17mm -> keyboard stuff:mustekala-2-2-17mm
- G***: footprint keyboard stuff:routa-logo-smaller -> keyboard stuff:routa-logo-new-4-11mm
- moved G*** 0.20 mm to (157.4, 118.5)
Other:
- board text removed: "4.5; 2.75"
