File: kicad/ver2.0/pcb-bottom-plate/choctopus44-bottom-plate.kicad_pcb (KiCad board)
At the start: 2 copper layers, 243.9 x 111.9 mm, 11 parts

Commit message: new gerbers etc
Parts:
- removed the G*** at (144.8, 108.7)
- removed the G*** at (68.5, 113.2)
- removed the H1 at (69.6, 63.8)
- removed the H1 at (144.7, 109.7)
- removed H12: H12, MountingHole:MountingHole_2.2mm_M2_ISO14580_Pad
- removed H13: H13, MountingHole:MountingHole_2.2mm_M2_ISO14580_Pad
- removed H14: H14, MountingHole:MountingHole_2.2mm_M2_ISO14580_Pad
- removed the H6 at (144.7, 154.5)
- removed the H8 at (89.6, 111.2)
- removed the H8 at (199.8, 111.2)
- added G***: LOGO, keyboard stuff:lonkerot-6-155mm, B.Cu at (148.7, 85.7)
- added G***: LOGO, keyboard stuff:routa-logo-new-4-11mm, B.Cu at (88.0, 98.3)
- added H1: H1, MountingHole:MountingHole_2.2mm_M2_ISO14580_Pad, F.Cu at (75.7, 45.3)
- added H6: H6, MountingHole:MountingHole_2.2mm_M2_ISO14580_Pad, F.Cu at (148.3, 98.7)
- added H6: H6, MountingHole:MountingHole_2.2mm_M2_ISO14580_Pad, F.Cu at (123.9, 51.8)
- added H6: H6, MountingHole:MountingHole_2.2mm_M2_ISO14580_Pad, F.Cu at (160.2, 60.0)
- added H6: H6, MountingHole:MountingHole_2.2mm_M2_ISO14580_Pad, F.Cu at (136.0, 61.2)
- added H6: H6, MountingHole:MountingHole_2.2mm_M2_ISO14580_Pad, F.Cu at (148.3, 143.5)
- added H8: H8, MountingHole:MountingHole_2.2mm_M2_ISO14580_Pad, F.Cu at (225.1, 96.2)
- added H8: H8, MountingHole:MountingHole_2.2mm_M2_ISO14580_Pad, B.Cu at (71.6, 96.2)
- moved H11 18.6 mm to (221.0, 45.3), turned to 10 degrees
Other:
- board size 243.9 x 111.9 mm -> 247.4 x 121.4 mm
- net class Default removed
- board text added: "Choctopus44v2 by Routa Keebs 2023 Loosely based on Reviung41 rev1.3 GH by gtips 2021"
- board text removed: "Choctopus44 [Prototype] Designed by Routa#1858/SlightHeadache 2021 Based on REVIUNG41 rev1.3 GH by gtips 2021"
